Commit message: Rename packages and add MoveIt & hardware
Refactor/rename packages and add MoveIt + hardware integration files.

- Renamed drago_pkg -> drago_description_pkg and updated CMakeLists, package.xml, launch files, URDF mesh paths, and config files accordingly.
- Renamed robot_hardware_interface -> drago_hardware_interface: updated includes, header guards, plugin.xml, package metadata, and source paths; added drago_hardware_interface/ros2_control.urdf.xacro to configure ros2_control with the hardware plugin.
- Added and updated MoveIt integration: drago_moveit_pkg changes include new/updated CMakeLists (added calibration_node), new demo and task launch scripts, new moveit.rviz and rviz backup, updated joint_limits.yaml (higher velocity/acceleration limits), and added controller/rviz/MoveIt dependencies in package.xml.
- Added a new drago_task_pkg skeleton (CMakeLists, package.xml, example task/source files).
- Misc: updated README, install rules, and timestamps; adjusted robot_state_publisher/rviz launch args to use new package names.

Purpose: reorganize package names for clearer separation (robot description vs other code), and add scaffolding for MoveIt, controllers, and the hardware interface for simulation/real-hardware integration.

File: Software/drago_description_pkg/urdf/drago.urdf (robot description, URDF)
Before this commit: robot Drago, 7 links, 6 joints
Links:
- link Effector_link: geometry collision mesh filename=package://drago_description_pkg/meshes/Effector_link.STL; visual mesh filename=package://drago_description_pkg/meshes/Effector_link.STL
- link Elbow_link: geometry collision mesh filename=package://drago_description_pkg/meshes/Elbow_link.STL; visual mesh filename=package://drago_description_pkg/meshes/Elbow_link.STL
- link Shoulder_link: geometry collision mesh filename=package://drago_description_pkg/meshes/Shoulder_link.STL; visual mesh filename=package://drago_description_pkg/meshes/Shoulder_link.STL
- link Waist_link: geometry collision mesh filename=package://drago_description_pkg/meshes/Waist_link.STL; visual mesh filename=package://drago_description_pkg/meshes/Waist_link.STL
- link Wrist_1_link: geometry collision mesh filename=package://drago_description_pkg/meshes/Wrist_1_link.STL; visual mesh filename=package://drago_description_pkg/meshes/Wrist_1_link.STL
- link Wrist_2_link: geometry collision mesh filename=package://drago_description_pkg/meshes/Wrist_2_link.STL; visual mesh filename=package://drago_description_pkg/meshes/Wrist_2_link.STL
- link base_link: geometry collision mesh filename=package://drago_description_pkg/meshes/base_link.STL; visual mesh filename=package://drago_description_pkg/meshes/base_link.STL

Commit message: Added a brand new gripper
URDF, control & hardware interface changes to feat the new gripper tool

File: Software/drago_description_pkg/urdf/drago.urdf (robot description, URDF)
Before this commit: robot Drago, 7 links, 6 joints
Links:
- added link Gripper_link, mass 0.0338622957317034; collision mesh filename=package://drago_description_pkg/meshes/Gripper_link.STL; visual mesh filename=package://drago_description_pkg/meshes/Gripper_link.STL
- added link Left_Claw_link, mass 0.00458904733917677; collision mesh filename=package://drago_description_pkg/meshes/Left_Claw_link.STL; visual mesh filename=package://drago_description_pkg/meshes/Left_Claw_link.STL
- added link Right_Claw_link, mass 0.00458904721552371; collision mesh filename=package://drago_description_pkg/meshes/Right_Claw_link.STL; visual mesh filename=package://drago_description_pkg/meshes/Right_Claw_link.STL
- link Effector_link: mass 0.00118783436629656 -> 0.0031625371291834
- link Elbow_link: mass 0.104178577887407 -> 0.0997434531792725
- link Shoulder_link: mass 0.0683062909364027 -> 0.0683063019704699
- link Waist_link: mass 0.114312274057208 -> 0.114312272517247
- link Wrist_1_link: mass 0.0380971171326554 -> 0.0364225917173961
- link Wrist_2_link: mass 0.0143322219516906 -> 0.0139246019270835
- link base_link: mass 0.150185390114133 -> 0.1474375874572
Joints:
- added joint Gripper_joint: type fixed, parent Effector_link, child Gripper_link, origin xyz=0.000766471836677465 0.00373197464508285 0.0551499896883955 rpy=0 0 0, axis 0 0 0
- added joint Left_Claw_joint: type prismatic, parent Gripper_link, child Left_Claw_link, origin xyz=0.022567 -0.0003 0 rpy=0 -1.5708 0, axis 0 0 1, limit lower=0 upper=0.013 effort=0 velocity=0
- added joint Right_Claw_joint: type prismatic, parent Gripper_link, child Right_Claw_link, origin xyz=-0.022433 -0.0003 0 rpy=3.1415 -1.5708 0, axis 0 0 1, limit lower=0 upper=0.013 effort=0 velocity=0
- joint Effector_joint: axis 1 0 0.0010354 -> 0 0 1; origin xyz=0.040844 -0.0051105 -0.0013078 rpy=0 0.0010354 0 -> xyz=0.0408435294675011 -0.00511048363110789 -0.00140782639546167 rpy=0 1.5707963267949 0
- joint Elbow_joint: axis 0.00103536403989601 0 -0.999999464010509 -> 0 0 -1; origin xyz=0 0.12 0 rpy=0.000730291763721768 0 -0.614305797905159 -> xyz=0 0.12 0 rpy=0 0 -0.559711205792866
- joint Shoulder_joint: axis 0.0012670059545015 0 -0.999999197347633 -> 0 0 -1; origin xyz=-0.0138993282947757 0.0103143963931036 0.04028 rpy=1.56990264699179 -0.614305609815112 0.000515109286944776 -> xyz=0.00470000000000012 -0.01391 0.0402799999999999 rpy=1.5707963267949 -0.559711205792866 1.5707963267949
- joint Waist_joint: origin xyz=0 0 0.06165 rpy=0 0 0 -> xyz=0 0.000299999804291295 0.0823428680948091 rpy=0 0 0
- joint Wrist_1_joint: axis 0.001035364039901 0 -0.999999464010509 -> -1 0 0; origin xyz=0.0943999494025927 -0.005 9.77383653464683E-05 rpy=0 1.5707963267949 0 -> xyz=0.0944000000000003 -0.00500000000000012 -0.0150000000000001 rpy=0 0 0
- joint Wrist_2_joint: limit lower=-1.57 upper=1.396 effort=1 velocity=3 -> lower=-1.57 upper=1.57 effort=1 velocity=3; origin xyz=-0.0013012254232319 0.0034038765092409 0.0208385964872179 rpy=-3.14159265358979 -1.56976096256998 3.14159265358979 -> xyz=0.0208399325599607 0.00340387650924096 0.00127964919234359 rpy=0 0 0

File: Software/drago_moveit_pkg/config/Drago.ros2_control.xacro (robot description, xacro)
@@ -5,10 +5,23 @@
         <ros2_control name="DragoSystem" type="system">
             <hardware>
-                <!-- By default, set up controllers for simulation. This won't work on real hardware -->
+                 <!-- By default, set up controllers for simulation. This won't work on real hardware -->
                 <!--<plugin>mock_components/GenericSystem</plugin>-->
-                <plugin>robot_hardware_interface/RobotHardwareInterface</plugin>
-                <param name="serial_port">/dev/ttyACM0</param>
+                <plugin>drago_hardware_interface/RobotHardwareInterface</plugin>
+                <param name="serial_port">/dev/ttyUSB0</param>
                 <param name="baud_rate">115200</param>
+                <param name="gripper_closed_servo_angle_deg">30.0</param>
             </hardware>
+            <joint name="Left_Claw_joint">
+                <command_interface name="position"/>
+                <state_interface name="position">
+                  <param name="initial_value">${initial_positions['Left_Claw_joint']}</param>
+                </state_interface>
+            </joint>
+            <joint name="Right_Claw_joint">
+                <command_interface name="position"/>
+                <state_interface name="position">
+                  <param name="initial_value">${initial_positions['Right_Claw_joint']}</param>
+                </state_interface>
+            </joint>
             <joint name="Waist_joint">
                 <command_interface name="position"/>

File: Software/drago_moveit_pkg/config/Drago.urdf.xacro (robot description, xacro)
@@ -3,5 +3,5 @@
     <xacro:arg name="initial_positions_file" default="initial_positions.yaml" />
     <!-- Import Drago urdf file -->
-    <xacro:include filename="$(find drago_pkg)/urdf/drago.urdf" />
+    <xacro:include filename="$(find drago_description_pkg)/urdf/drago.urdf" />
     <!-- Import control_xacro -->
     <xacro:include filename="Drago.ros2_control.xacro" />
